File: kicad/kinetis.sch (KiCad schematic (older format))
At the start: 70 parts, among them J1 CONN_01X16, J2 CONN_01X16, J3 CONN_01X16, J4 CONN_01X16, J5 USB_Micro_B, J6 FTDI_Connector, J7 JLink_SWD_20pin, SW1 SPST, SW2 SPST, SW3 SPST, SW4 SPST, SW5 SPST, SW6 DPDT, U1 MKL16Z64VLH4, U2 LM1117-ADJ, Y1 12.000 MHz

Commit message: Added 1x16 footprint. Added 'shield' pin to USB connector.
Parts:
- J1, J2, J3, J4: footprint (none) -> Header_0.1in_1x16
Connections:
- wire segments 299 -> 301
Other:
- moved on the sheet: J5
Changed lines of the file:
@@
 Text Notes 14400 6550 0    60   ~ 0
 Header for 6-pin Sparkfun\nor Adafruit USB-UART cable.
-Text Notes 12600 6900 0    60   ~ 0
+Text Notes 12450 6850 0    60   ~ 0
 USB Micro-B connector.\nUsed for power only.
 $Comp
@@
 L USB_Micro_B J5
 U 1 1 58C71BB0
-P 12850 5900
-F 0 "J5" H 12650 6350 60  0000 C CNN
-F 1 "USB_Micro_B" H 12875 6250 60  0000 C CNN
-F 2 "" H 13250 5850 60  0001 C CNN
-F 3 "" H 13250 5850 60  0001 C CNN
-F 4 "Amphenol FCI" H 12750 6450 60  0001 C CNN "Manufacturer"
-F 5 "10118192-0001LF" H 12750 6550 60  0001 C CNN "Manufacturer PN"
-	1    12850 5900
+P 12450 5650
+F 0 "J5" H 12500 5810 60  0000 C CNN
+F 1 "USB_Micro_B" H 12730 5730 60  0000 C CNN
+F 2 "" H 12850 5600 60  0001 C CNN
+F 3 "" H 12850 5600 60  0001 C CNN
+F 4 "Amphenol FCI" H 12350 6200 60  0001 C CNN "Manufacturer"
+F 5 "10118192-0001LF" H 12350 6300 60  0001 C CNN "Manufacturer PN"
+	1    12450 5650
 	1    0    0    -1
 $EndComp
@@
 	13600 5800 13600 5750
 Wire Wire Line
-	13050 5800 13600 5800
-Wire Wire Line
-	13050 5900 13600 5900
-Wire Wire Line
-	13050 5700 13200 5700
+	13000 5800 13600 5800
+Wire Wire Line
+	13000 5900 13600 5900
+Wire Wire Line
+	13000 5700 13200 5700
 Wire Wire Line
 	13200 5700 13200 5400
@@
 Connection ~ 15150 3700
 Wire Wire Line
-	13050 6000 13250 6000
+	13000 6000 13250 6000
 Wire Wire Line
 	13250 6000 13250 6050
@@
 F 0 "J1" H 3300 3150 50  0000 C CNN
 F 1 "CONN_01X16" H 3100 3050 50  0000 C CNN
-F 2 "" H 3300 2150 50  0001 C CNN
+F 2 "Header_0.1in_1x16" H 3300 2150 50  0001 C CNN
 F 3 "" H 3300 3000 50  0001 C CNN
 F 4 "Sullins" H 3375 3175 60  0001 C CNN "Manufacturer"
@@
 F 0 "J2" H 3300 5250 50  0000 C CNN
 F 1 "CONN_01X16" H 3100 5150 50  0000 C CNN
-F 2 "" H 3300 4250 50  0001 C CNN
+F 2 "Header_0.1in_1x16" H 3300 4250 50  0001 C CNN
 F 3 "" H 3300 5100 50  0001 C CNN
 F 4 "Sullins" H 3375 5275 60  0001 C CNN "Manufacturer"
@@
 F 0 "J3" H 3300 7350 50  0000 C CNN
 F 1 "CONN_01X16" H 3100 7250 50  0000 C CNN
-F 2 "" H 3300 6350 50  0001 C CNN
+F 2 "Header_0.1in_1x16" H 3300 6350 50  0001 C CNN
 F 3 "" H 3300 7200 50  0001 C CNN
 F 4 "Sullins" H 3375 7375 60  0001 C CNN "Manufacturer"
@@
 F 0 "J4" H 3300 9450 50  0000 C CNN
 F 1 "CONN_01X16" H 3100 9350 50  0000 C CNN
-F 2 "" H 3300 8450 50  0001 C CNN
+F 2 "Header_0.1in_1x16" H 3300 8450 50  0001 C CNN
 F 3 "" H 3300 9300 50  0001 C CNN
 F 4 "Sullins" H 3375 9475 60  0001 C CNN "Manufacturer"
@@
 	0    1    1    0
 $EndComp
+Wire Wire Line
+	13000 6100 13050 6100
+Wire Wire Line
+	13000 6250 13050 6250
+Connection ~ 13050 6250
 $EndSCHEMATC

Commit message: Added footprint for Micro-USB connector.
Parts:
- J5: footprint (none) -> 10118192-0001LF
Changed lines of the file:
@@
 F 0 "J5" H 12500 5810 60  0000 C CNN
 F 1 "USB_Micro_B" H 12730 5730 60  0000 C CNN
-F 2 "" H 12850 5600 60  0001 C CNN
+F 2 "10118192-0001LF" H 12850 5600 60  0001 C CNN
 F 3 "" H 12850 5600 60  0001 C CNN
 F 4 "Amphenol FCI" H 12350 6200 60  0001 C CNN "Manufacturer"

Commit message: Added footprints for 1x6 and 2x10 headers.
This commit adds footprints for the FTDI header (1x6, 0.1") and
the J-Link header (2x10, 0.1", shrouded). The schematic was also
updated to match.
Parts:
- J6: footprint (none) -> Header_0.1in_1x6
- J7: footprint (none) -> Header_Shrouded_0.1in_2x10
Changed lines of the file:
@@
 F 0 "J6" H 14425 6575 50  0000 C CNN
 F 1 "FTDI_Connector" H 14675 6500 50  0000 C CNN
-F 2 "" H 14650 6050 50  0001 C CNN
+F 2 "Header_0.1in_1x6" H 14650 6050 50  0001 C CNN
 F 3 "" H 14650 6050 50  0001 C CNN
 F 4 "Sullins" H 14525 6675 60  0001 C CNN "Manufacturer"
@@
 F 0 "J7" H 14675 8450 50  0000 C CNN
 F 1 "JLink_SWD_20pin" H 14950 8375 50  0000 C CNN
-F 2 "" H 14900 6400 50  0001 C CNN
+F 2 "Header_Shrouded_0.1in_2x10" H 14900 6400 50  0001 C CNN
 F 3 "" H 14900 6400 50  0001 C CNN
 F 4 "On Shore" H 14775 8550 60  0001 C CNN "Manufacturer"
