File: kicad/kinetis.sch (KiCad schematic (older format))
At the start: 70 parts, among them J1 CONN_01X16, J2 CONN_01X16, J3 CONN_01X16, J4 CONN_01X16, J5 USB_Micro_B, J6 FTDI_Connector, J7 JLink_SWD_20pin, SW1 SPST, SW2 SPST, SW3 SPST, SW4 SPST, SW5 SPST, SW6 DPDT, U1 MKL16Z64VLH4, U2 LM1117-ADJ, Y1 12.000 MHz

Commit message: Tweaked DPDT schematic symbol, and complete footprints.
This commit adds the final two footprints, and also tweaks the pin
ordering of the DPDT switch.

The footprints should still be reviewed, but they all look good at
a glance.
Parts:
- SW1, SW2, SW3, SW4, SW5: footprint (none) -> PTS645_SMT
- SW6: footprint (none) -> GF-126-0159; Manufacturer (none) -> CW Industries; Manufacturer PN (none) -> GF-126-0159

Commit message: Fixed schematic footprint callouts
Parts:
- D5, D6, D7, D8: footprint SOD-123F -> SOD_123F
- U1: footprint LFQP-64 -> QFP_64
Changed lines of the file:
@@
 F 0 "D8" V 14450 2700 50  0000 C CNN
 F 1 "400mV@0.5A" V 14350 2850 50  0000 C CNN
-F 2 "SOD-123F" H 14400 2550 50  0001 C CNN
+F 2 "SOD_123F" H 14400 2550 50  0001 C CNN
 F 3 "" H 14300 2750 50  0001 C CNN
 F 4 "ON Semi" H 14400 2850 60  0001 C CNN "Manufacturer"
@@
 F 0 "D5" H 12650 2250 50  0000 L CNN
 F 1 "400mV@0.5A" H 12450 2150 50  0000 L CNN
-F 2 "SOD-123F" H 12700 2000 50  0001 C CNN
+F 2 "SOD_123F" H 12700 2000 50  0001 C CNN
 F 3 "" H 12600 2200 50  0001 C CNN
 F 4 "ON Semi" H 12700 2300 60  0001 C CNN "Manufacturer"
@@
 F 0 "D6" H 12650 2650 50  0000 L CNN
 F 1 "400mV@0.5A" H 12450 2550 50  0000 L CNN
-F 2 "SOD-123F" H 12700 2400 50  0001 C CNN
+F 2 "SOD_123F" H 12700 2400 50  0001 C CNN
 F 3 "" H 12600 2600 50  0001 C CNN
 F 4 "ON Semi" H 12700 2700 60  0001 C CNN "Manufacturer"
@@
 F 0 "D7" H 12650 3050 50  0000 L CNN
 F 1 "400mV@0.5A" H 12450 2950 50  0000 L CNN
-F 2 "SOD-123F" H 12700 2800 50  0001 C CNN
+F 2 "SOD_123F" H 12700 2800 50  0001 C CNN
 F 3 "" H 12600 3000 50  0001 C CNN
 F 4 "ON Semi" H 12700 3100 60  0001 C CNN "Manufacturer"
@@
 F 0 "U1" H 4950 7750 60  0000 C CNN
 F 1 "MKL16Z64VLH4" H 5200 7650 60  0000 C CNN
-F 2 "LFQP-64" H 4925 6775 60  0001 C CNN
+F 2 "QFP_64" H 4925 6775 60  0001 C CNN
 F 3 "" H 4925 6775 60  0001 C CNN
 F 4 "NXP" H 5000 7850 60  0001 C CNN "Manufacturer"
@@
 F 0 "U1" H 4950 5650 60  0000 C CNN
 F 1 "MKL16Z64VLH4" H 5200 5550 60  0000 C CNN
-F 2 "LFQP-64" H 4925 4675 60  0001 C CNN
+F 2 "QFP_64" H 4925 4675 60  0001 C CNN
 F 3 "" H 4925 4675 60  0001 C CNN
 F 4 "NXP" H 5000 5750 60  0001 C CNN "Manufacturer"
@@
 F 0 "U1" H 4950 3550 60  0000 C CNN
 F 1 "MKL16Z64VLH4" H 5200 3450 60  0000 C CNN
-F 2 "LFQP-64" H 4925 2575 60  0001 C CNN
+F 2 "QFP_64" H 4925 2575 60  0001 C CNN
 F 3 "" H 4925 2575 60  0001 C CNN
 F 4 "NXP" H 5000 3650 60  0001 C CNN "Manufacturer"
@@
 F 0 "U1" H 4950 1450 60  0000 C CNN
 F 1 "MKL16Z64VLH4" H 5200 1350 60  0000 C CNN
-F 2 "LFQP-64" H 4925 475 60  0001 C CNN
+F 2 "QFP_64" H 4925 475 60  0001 C CNN
 F 3 "" H 4925 475 60  0001 C CNN
 F 4 "NXP" H 5000 1550 60  0001 C CNN "Manufacturer"

Commit message: Selected custom library for all components.
Parts:
- C1, C10, C12, C2, C3, C4, C5, C6, C7, C9: footprint SM_0603 -> custom_footprints:SM_0603
- C11, C8: footprint SM_1206 -> custom_footprints:SM_1206
- D1, D2, D3, D4, D9: footprint D_0805 -> custom_footprints:D_0805
- D5, D6, D7, D8: footprint SOD_123F -> custom_footprints:SOD_123F
- F1: footprint SM_1812 -> custom_footprints:SM_1812
- J1, J2, J3, J4: footprint Header_0.1in_1x16 -> custom_footprints:Header_0.1in_1x16
- J5: footprint 10118192-0001LF -> custom_footprints:10118192-0001LF
- J6: footprint Header_0.1in_1x6 -> custom_footprints:Header_0.1in_1x6
- J7: footprint Header_Shrouded_0.1in_2x10 -> custom_footprints:Header_Shrouded_0.1in_2x10
- R1, R10, R11, R12, R13, R14, R15, R16, R17, R18, R19, R2, R20, R21, R22, R23, R24, R25, R26, R27, R28, R29, R3, R30, R31, R32, R4, R5, R6, R7, R8, R9: footprint SM_0805 -> custom_footprints:SM_0805
- SW1, SW2, SW3, SW4, SW5: footprint PTS645_SMT -> custom_footprints:PTS645_SMT
- SW6: footprint GF-126-0159 -> custom_footprints:GF-126-0159
- U1: footprint QFP_64 -> custom_footprints:QFP_64
- U2: footprint SOT-223 -> custom_footprints:SOT_223_3
- Y1: footprint SM_HC49US -> custom_footprints:SM_HC49US

Commit message: Misc pin tweaks. Lots more routing.
Parts:
- removed R15, R18, R19, R20: 200, custom_footprints:SM_0805, symbol R
- added C13, C14, C15, C16: 0.1uF, custom_footprints:SM_0603, symbol C
- R13, R14, R5, R6: value 0.1 -> 200
Connections:
- wire segments 301 -> 309
Other:
- moved on the sheet: R13, R14, R3, R4

Commit message: Added mounting holes. Moved stuff. More routing.
This commit adds 4-40 mounting holes to the design, and shoves
a bunch of stuff around to make room for them. It also moves
the DPDT switch to ignore the secondary switch pole, in order to make
some routing space.
Parts:
- added M1, M2, M3, M4: #4-40 Mounting Hole, custom_footprints:4_40_Hole, symbol HOLE
- J7: Manufacturer On Shore -> CNC Tech; Manufacturer PN 302-S201 -> 3020-20-0100-00
Connections:
- wire segments 309 -> 312
- no-connect marks 13 -> 16
Other:
- moved on the sheet: F1, R23
Changed lines of the file:
@@
 L GND #PWR07
 U 1 1 58C4006A
-P 13250 2750
-F 0 "#PWR07" H 13250 2500 50  0001 C CNN
-F 1 "GND" H 13250 2600 50  0000 C CNN
-F 2 "" H 13250 2750 50  0001 C CNN
-F 3 "" H 13250 2750 50  0001 C CNN
-	1    13250 2750
+P 13225 2750
+F 0 "#PWR07" H 13225 2500 50  0001 C CNN
+F 1 "GND" H 13225 2600 50  0000 C CNN
+F 2 "" H 13225 2750 50  0001 C CNN
+F 3 "" H 13225 2750 50  0001 C CNN
+	1    13225 2750
 	1    0    0    -1
 $EndComp
@@
 L PTC F1
 U 1 1 58C52C19
-P 14200 1950
-F 0 "F1" V 14000 1900 50  0000 C CNN
-F 1 "500mA PTC" V 14100 1850 50  0000 L CNN
-F 2 "custom_footprints:SM_1812" H 14250 1750 50  0001 L CNN
-F 3 "" V 14100 1950 50  0001 C CNN
-F 4 "Bel Fuse" V 13900 2000 60  0001 C CNN "Manufacturer"
-F 5 "0ZCG0050FF2C" V 14000 2000 60  0001 C CNN "Manufacturer PN"
-	1    14200 1950
+P 14175 1950
+F 0 "F1" V 13995 1895 50  0000 C CNN
+F 1 "500mA PTC" V 14075 1845 50  0000 L CNN
+F 2 "custom_footprints:SM_1812" H 14225 1750 50  0001 L CNN
+F 3 "" V 14075 1950 50  0001 C CNN
+F 4 "Bel Fuse" V 13875 2000 60  0001 C CNN "Manufacturer"
+F 5 "0ZCG0050FF2C" V 13975 2000 60  0001 C CNN "Manufacturer PN"
+	1    14175 1950
 	0    1    1    0
 $EndComp
@@
 L R R23
 U 1 1 58C5951A
-P 13250 2550
-F 0 "R23" V 13200 2350 50  0000 L CNN
-F 1 "200" V 13300 2350 50  0000 L CNN
-F 2 "custom_footprints:SM_0805" V 13180 2550 50  0001 C CNN
-F 3 "" H 13250 2750 50  0001 C CNN
-F 4 "Yageo" H 13250 2850 60  0001 C CNN "Manufacturer"
-F 5 "RC0805FR-07200RL" H 13250 2950 60  0001 C CNN "Manufacturer PN"
-	1    13250 2550
+P 13225 2550
+F 0 "R23" V 13175 2350 50  0000 L CNN
+F 1 "200" V 13275 2350 50  0000 L CNN
+F 2 "custom_footprints:SM_0805" V 13155 2550 50  0001 C CNN
+F 3 "" H 13225 2750 50  0001 C CNN
+F 4 "Yageo" H 13225 2850 60  0001 C CNN "Manufacturer"
+F 5 "RC0805FR-07200RL" H 13225 2950 60  0001 C CNN "Manufacturer PN"
+	1    13225 2550
 	0    1    1    0
 $EndComp
@@
 F 2 "custom_footprints:Header_Shrouded_0.1in_2x10" H 14900 6400 50  0001 C CNN
 F 3 "" H 14900 6400 50  0001 C CNN
-F 4 "On Shore" H 14775 8550 60  0001 C CNN "Manufacturer"
-F 5 "302-S201" H 14775 8650 60  0001 C CNN "Manufacturer PN"
+F 4 "CNC Tech" H 14775 8550 60  0001 C CNN "Manufacturer"
+F 5 "3020-20-0100-00" H 14775 8650 60  0001 C CNN "Manufacturer PN"
 	1    14900 7600
 	1    0    0    -1
@@
 $EndComp
 $Comp
-L DPDT SW6
-U 1 1 58C63D13
-P 13575 2150
-F 0 "SW6" H 13740 1770 60  0000 C CNN
-F 1 "DPDT" H 13720 1850 60  0000 C CNN
-F 2 "custom_footprints:GF-126-0159" H 13575 2025 60  0001 C CNN
-F 3 "" H 13575 2025 60  0001 C CNN
-F 4 "CW Industries" H 13400 2675 60  0001 C CNN "Manufacturer"
-F 5 "GF-126-0159" H 13400 2775 60  0001 C CNN "Manufacturer PN"
-	1    13575 2150
-	-1   0    0    1
-$EndComp
-$Comp
 L C C13
 U 1 1 58CB1D2D
@@
 	12450 2400 12550 2400
 Wire Wire Line
-	12850 2400 13000 2400
-Wire Wire Line
-	12850 2000 13275 2000
+	12850 2400 12975 2400
 Wire Wire Line
 	12450 2800 12550 2800
 Wire Wire Line
-	13000 2800 12850 2800
-Wire Wire Line
-	13000 2000 13000 2800
-Connection ~ 13000 2400
-Wire Wire Line
-	13275 2100 13250 2100
-Wire Wire Line
-	13250 2100 13250 2400
-Wire Wire Line
-	13250 2350 13275 2350
-Wire Wire Line
-	13275 2250 13200 2250
-Wire Wire Line
-	13200 2250 13200 2000
-Connection ~ 13200 2000
-Connection ~ 13000 2000
-Connection ~ 13250 2350
-Wire Wire Line
-	13925 1950 14050 1950
-Wire Wire Line
-	14000 1950 14000 2200
-Wire Wire Line
-	14000 2200 13925 2200
-Connection ~ 14000 1950
+	12975 2800 12850 2800
+Wire Wire Line
+	12975 2000 12975 2800
+Connection ~ 12975 2400
+Connection ~ 12975 2000
 Wire Wire Line
 	15500 7100 15500 7800
@@
 Connection ~ 14400 1950
 Wire Wire Line
-	14350 1950 15150 1950
-Wire Wire Line
-	13250 2750 13250 2700
+	14325 1950 15150 1950
+Wire Wire Line
+	13225 2750 13225 2700
 Wire Wire Line
 	9650 5275 9650 5375
@@
 Wire Wire Line
 	1600 8900 1900 8900
+$Comp
+L HOLE M1
+U 1 1 58CB7CC4
+P 10300 8550
+F 0 "M1" H 10473 8596 50  0000 L CNN
+F 1 "#4-40 Mounting Hole" H 10473 8505 50  0000 L CNN
+F 2 "custom_footprints:4_40_Hole" H 10300 8550 50  0001 C CNN
+F 3 "" H 10300 8750 50  0001 C CNN
+F 4 "(none)" H 10300 9025 60  0001 C CNN "Manufacturer"
+F 5 "(none)" H 10300 8900 60  0001 C CNN "Manufacturer PN"
+	1    10300 8550
+	1    0    0    -1
+$EndComp
+$Comp
+L HOLE M2
+U 1 1 58CB7E94
+P 10300 8900
+F 0 "M2" H 10473 8946 50  0000 L CNN
+F 1 "#4-40 Mounting Hole" H 10473 8855 50  0000 L CNN
+F 2 "custom_footprints:4_40_Hole" H 10300 8900 50  0001 C CNN
+F 3 "" H 10300 9100 50  0001 C CNN
+F 4 "(none)" H 10300 9375 60  0001 C CNN "Manufacturer"
+F 5 "(none)" H 10300 9250 60  0001 C CNN "Manufacturer PN"
+	1    10300 8900
+	1    0    0    -1
+$EndComp
+$Comp
+L HOLE M3
+U 1 1 58CB7F7E
+P 10300 9250
+F 0 "M3" H 10473 9296 50  0000 L CNN
+F 1 "#4-40 Mounting Hole" H 10473 9205 50  0000 L CNN
+F 2 "custom_footprints:4_40_Hole" H 10300 9250 50  0001 C CNN
+F 3 "" H 10300 9450 50  0001 C CNN
+F 4 "(none)" H 10300 9725 60  0001 C CNN "Manufacturer"
+F 5 "(none)" H 10300 9600 60  0001 C CNN "Manufacturer PN"
+	1    10300 9250
+	1    0    0    -1
+$EndComp
+$Comp
+L HOLE M4
+U 1 1 58CB8044
+P 10300 9600
+F 0 "M4" H 10473 9646 50  0000 L CNN
+F 1 "#4-40 Mounting Hole" H 10473 9555 50  0000 L CNN
+F 2 "custom_footprints:4_40_Hole" H 10300 9600 50  0001 C CNN
+F 3 "" H 10300 9800 50  0001 C CNN
+F 4 "(none)" H 10300 10075 60  0001 C CNN "Manufacturer"
+F 5 "(none)" H 10300 9950 60  0001 C CNN "Manufacturer PN"
+	1    10300 9600
+	1    0    0    -1
+$EndComp
+$Comp
+L GND #PWR040
+U 1 1 58CB8882
+P 10050 9650
+F 0 "#PWR040" H 10050 9400 50  0001 C CNN
+F 1 "GND" H 10050 9500 50  0000 C CNN
+F 2 "" H 10050 9650 50  0001 C CNN
+F 3 "" H 10050 9650 50  0001 C CNN
+	1    10050 9650
+	-1   0    0    -1
+$EndComp
+Wire Wire Line
+	10100 9600 10050 9600
+Wire Wire Line
+	10050 9600 10050 9650
+$Comp
+L GND #PWR041
+U 1 1 58CB8BE9
+P 10050 9300
+F 0 "#PWR041" H 10050 9050 50  0001 C CNN
+F 1 "GND" H 10050 9150 50  0000 C CNN
+F 2 "" H 10050 9300 50  0001 C CNN
+F 3 "" H 10050 9300 50  0001 C CNN
+	1    10050 9300
+	-1   0    0    -1
+$EndComp
+$Comp
+L GND #PWR042
+U 1 1 58CB8C8E
+P 10050 8950
+F 0 "#PWR042" H 10050 8700 50  0001 C CNN
+F 1 "GND" H 10050 8800 50  0000 C CNN
+F 2 "" H 10050 8950 50  0001 C CNN
+F 3 "" H 10050 8950 50  0001 C CNN
+	1    10050 8950
+	-1   0    0    -1
+$EndComp
+$Comp
+L GND #PWR043
+U 1 1 58CB8D80
+P 10050 8600
+F 0 "#PWR043" H 10050 8350 50  0001 C CNN
+F 1 "GND" H 10050 8450 50  0000 C CNN
+F 2 "" H 10050 8600 50  0001 C CNN
+F 3 "" H 10050 8600 50  0001 C CNN
+	1    10050 8600
+	-1   0    0    -1
+$EndComp
+Wire Wire Line
+	10100 8550 10050 8550
+Wire Wire Line
+	10050 8550 10050 8600
+Wire Wire Line
+	10100 8900 10050 8900
+Wire Wire Line
+	10050 8900 10050 8950
+Wire Wire Line
+	10100 9250 10050 9250
+Wire Wire Line
+	10050 9250 10050 9300
+Wire Notes Line
+	9900 8300 11400 8300
+Wire Notes Line
+	9900 9900 11400 9900
+Wire Notes Line
+	9900 8300 9900 9900
+Wire Notes Line
+	11400 9900 11400 8300
+$Comp
+L DPDT SW6
+U 1 1 58CBA12A
+P 13600 2200
+F 0 "SW6" H 13430 2640 60  0000 C CNN
+F 1 "DPDT" H 13450 2550 60  0000 C CNN
+F 2 "custom_footprints:GF-126-0159" H 13600 2375 60  0001 C CNN
+F 3 "" H 13600 2375 60  0001 C CNN
+F 4 "CW Industries" H 13475 2725 60  0001 C CNN "Manufacturer"
+F 5 "GF-126-0159" H 13475 2825 60  0001 C CNN "Manufacturer PN"
+	1    13600 2200
+	1    0    0    -1
+$EndComp
+Wire Wire Line
+	13950 1950 14025 1950
+Wire Wire Line
+	12850 2000 13300 2000
+Wire Wire Line
+	13300 2100 13225 2100
+Wire Wire Line
+	13225 2100 13225 2400
+NoConn ~ 13300 2250
+NoConn ~ 13300 2350
+NoConn ~ 13950 2200
 $EndSCHEMATC

Commit message: Fixed library gaff
Changed lines of the file:
@@
 Wire Notes Line
 	11400 9900 11400 8300
-$Comp
-L DPDT SW6
-U 1 1 58CBA12A
-P 13600 2200
-F 0 "SW6" H 13430 2640 60  0000 C CNN
-F 1 "DPDT" H 13450 2550 60  0000 C CNN
-F 2 "custom_footprints:GF-126-0159" H 13600 2375 60  0001 C CNN
-F 3 "" H 13600 2375 60  0001 C CNN
-F 4 "CW Industries" H 13475 2725 60  0001 C CNN "Manufacturer"
-F 5 "GF-126-0159" H 13475 2825 60  0001 C CNN "Manufacturer PN"
-	1    13600 2200
-	1    0    0    -1
-$EndComp
 Wire Wire Line
 	13950 1950 14025 1950
@@
 NoConn ~ 13300 2350
 NoConn ~ 13950 2200
+$Comp
+L DPDT SW6
+U 1 1 58CBE31C
+P 13600 2200
+F 0 "SW6" H 13430 2650 60  0000 C CNN
+F 1 "DPDT" H 13450 2560 60  0000 C CNN
+F 2 "custom_footprints:GF-126-0159" H 13600 2375 60  0001 C CNN
+F 3 "" H 13600 2375 60  0001 C CNN
+F 4 "CW Industries" H 13475 2725 60  0001 C CNN "Manufacturer"
+F 5 "GF-126-0159" H 13475 2825 60  0001 C CNN "Manufacturer PN"
+	1    13600 2200
+	1    0    0    -1
+$EndComp
 $EndSCHEMATC

Commit message: Reconciled +3.3V and +3V3 nets
Changed lines of the file:
@@
 LED[0]
 $Comp
-L +3.3V #PWR014
-U 1 1 58C430A8
-P 8500 5550
-F 0 "#PWR014" H 8500 5400 50  0001 C CNN
-F 1 "+3.3V" H 8500 5690 50  0000 C CNN
-F 2 "" H 8500 5550 50  0001 C CNN
-F 3 "" H 8500 5550 50  0001 C CNN
-	1    8500 5550
-	1    0    0    -1
-$EndComp
-$Comp
-L GND #PWR015
+L GND #PWR014
 U 1 1 58C43C9E
 P 8500 6000
-F 0 "#PWR015" H 8500 5750 50  0001 C CNN
+F 0 "#PWR014" H 8500 5750 50  0001 C CNN
 F 1 "GND" H 8500 5850 50  0000 C CNN
 F 2 "" H 8500 6000 50  0001 C CNN
@@
 $EndComp
 $Comp
-L GND #PWR016
+L GND #PWR015
 U 1 1 58C49E1A
 P 8400 6950
-F 0 "#PWR016" H 8400 6700 50  0001 C CNN
+F 0 "#PWR015" H 8400 6700 50  0001 C CNN
 F 1 "GND" H 8400 6800 50  0000 C CNN
 F 2 "" H 8400 6950 50  0001 C CNN
@@
 $EndComp
 $Comp
-L +3.3V #PWR017
-U 1 1 58C4A60D
-P 7850 3450
-F 0 "#PWR017" H 7850 3300 50  0001 C CNN
-F 1 "+3.3V" H 7850 3590 50  0000 C CNN
-F 2 "" H 7850 3450 50  0001 C CNN
-F 3 "" H 7850 3450 50  0001 C CNN
-	1    7850 3450
-	1    0    0    -1
-$EndComp
-$Comp
-L GND #PWR018
+L GND #PWR016
 U 1 1 58C4A619
 P 7850 3900
-F 0 "#PWR018" H 7850 3650 50  0001 C CNN
+F 0 "#PWR016" H 7850 3650 50  0001 C CNN
 F 1 "GND" H 7850 3750 50  0000 C CNN
 F 2 "" H 7850 3900 50  0001 C CNN
@@
 $EndComp
 $Comp
-L GND #PWR019
+L GND #PWR017
 U 1 1 58C4A7A4
 P 7750 4850
-F 0 "#PWR019" H 7750 4600 50  0001 C CNN
+F 0 "#PWR017" H 7750 4600 50  0001 C CNN
 F 1 "GND" H 7750 4700 50  0000 C CNN
 F 2 "" H 7750 4850 50  0001 C CNN
@@
 $EndComp
 $Comp
-L +3.3V #PWR020
-U 1 1 58C4AF8C
-P 9550 1350
-F 0 "#PWR020" H 9550 1200 50  0001 C CNN
-F 1 "+3.3V" H 9550 1490 50  0000 C CNN
-F 2 "" H 9550 1350 50  0001 C CNN
-F 3 "" H 9550 1350 50  0001 C CNN
-	1    9550 1350
-	1    0    0    -1
-$EndComp
-$Comp
-L GND #PWR021
+L GND #PWR018
 U 1 1 58C4AF98
 P 9550 1800
-F 0 "#PWR021" H 9550 1550 50  0001 C CNN
+F 0 "#PWR018" H 9550 1550 50  0001 C CNN
 F 1 "GND" H 9550 1650 50  0000 C CNN
 F 2 "" H 9550 1800 50  0001 C CNN
@@
 $EndComp
 $Comp
-L +3.3V #PWR022
-U 1 1 58C4B093
-P 9100 1600
-F 0 "#PWR022" H 9100 1450 50  0001 C CNN
-F 1 "+3.3V" H 9100 1740 50  0000 C CNN
-F 2 "" H 9100 1600 50  0001 C CNN
-F 3 "" H 9100 1600 50  0001 C CNN
-	1    9100 1600
-	1    0    0    -1
-$EndComp
-$Comp
-L GND #PWR023
+L GND #PWR019
 U 1 1 58C4B09F
 P 9100 2050
-F 0 "#PWR023" H 9100 1800 50  0001 C CNN
+F 0 "#PWR019" H 9100 1800 50  0001 C CNN
 F 1 "GND" H 9100 1900 50  0000 C CNN
 F 2 "" H 9100 2050 50  0001 C CNN
@@
 $EndComp
 $Comp
-L +3.3V #PWR024
-U 1 1 58C4B1A4
-P 8650 1850
-F 0 "#PWR024" H 8650 1700 50  0001 C CNN
-F 1 "+3.3V" H 8650 1990 50  0000 C CNN
-F 2 "" H 8650 1850 50  0001 C CNN
-F 3 "" H 8650 1850 50  0001 C CNN
-	1    8650 1850
-	1    0    0    -1
-$EndComp
-$Comp
-L GND #PWR025
+L GND #PWR020
 U 1 1 58C4B1B0
 P 8650 2300
-F 0 "#PWR025" H 8650 2050 50  0001 C CNN
+F 0 "#PWR020" H 8650 2050 50  0001 C CNN
 F 1 "GND" H 8650 2150 50  0000 C CNN
 F 2 "" H 8650 2300 50  0001 C CNN
@@
 $EndComp
 $Comp
-L GND #PWR026
+L GND #PWR021
 U 1 1 58C4D12C
 P 8300 2350
-F 0 "#PWR026" H 8300 2100 50  0001 C CNN
+F 0 "#PWR021" H 8300 2100 50  0001 C CNN
 F 1 "GND" H 8300 2200 50  0000 C CNN
 F 2 "" H 8300 2350 50  0001 C CNN
@@
 NoConn ~ 14500 7100
 $Comp
-L +3.3V #PWR027
+L +3.3V #PWR022
 U 1 1 58C50449
 P 13550 7600
-F 0 "#PWR027" H 13550 7450 50  0001 C CNN
+F 0 "#PWR022" H 13550 7450 50  0001 C CNN
 F 1 "+3.3V" H 13550 7740 50  0000 C CNN
 F 2 "" H 13550 7600 50  0001 C CNN
@@
 $EndComp
 $Comp
-L +3.3V #PWR028
+L +3.3V #PWR023
 U 1 1 58C5CAA0
 P 9400 7050
-F 0 "#PWR028" H 9400 6900 50  0001 C CNN
+F 0 "#PWR023" H 9400 6900 50  0001 C CNN
 F 1 "+3.3V" H 9400 7190 50  0000 C CNN
 F 2 "" H 9400 7050 50  0001 C CNN
@@
 $EndComp
 $Comp
-L GND #PWR029
+L GND #PWR024
 U 1 1 58C5CAB2
 P 10100 7500
-F 0 "#PWR029" H 10100 7250 50  0001 C CNN
+F 0 "#PWR024" H 10100 7250 50  0001 C CNN
 F 1 "GND" H 10100 7350 50  0000 C CNN
 F 2 "" H 10100 7500 50  0001 C CNN
@@
 SW[W]
 $Comp
-L +3.3V #PWR030
+L +3.3V #PWR025
 U 1 1 58C60AB3
 P 10800 7050
-F 0 "#PWR030" H 10800 6900 50  0001 C CNN
+F 0 "#PWR025" H 10800 6900 50  0001 C CNN
 F 1 "+3.3V" H 10800 7190 50  0000 C CNN
 F 2 "" H 10800 7050 50  0001 C CNN
@@
 $EndComp
 $Comp
-L GND #PWR031
+L GND #PWR026
 U 1 1 58C60AC5
 P 11500 7500
-F 0 "#PWR031" H 11500 7250 50  0001 C CNN
+F 0 "#PWR026" H 11500 7250 50  0001 C CNN
 F 1 "GND" H 11500 7350 50  0000 C CNN
 F 2 "" H 11500 7500 50  0001 C CNN
@@
 SW[S]
 $Comp
-L +3.3V #PWR032
+L +3.3V #PWR027
 U 1 1 58C60CB4
 P 9400 6350
-F 0 "#PWR032" H 9400 6200 50  0001 C CNN
+F 0 "#PWR027" H 9400 6200 50  0001 C CNN
 F 1 "+3.3V" H 9400 6490 50  0000 C CNN
 F 2 "" H 9400 6350 50  0001 C CNN
@@
 $EndComp
 $Comp
-L GND #PWR033
+L GND #PWR028
 U 1 1 58C60CC6
 P 10100 6800
-F 0 "#PWR033" H 10100 6550 50  0001 C CNN
+F 0 "#PWR028" H 10100 6550 50  0001 C CNN
 F 1 "GND" H 10100 6650 50  0000 C CNN
 F 2 "" H 10100 6800 50  0001 C CNN
@@
 SW[N]
 $Comp
-L +3.3V #PWR034
+L +3.3V #PWR029
 U 1 1 58C60CD9
 P 10800 6350
-F 0 "#PWR034" H 10800 6200 50  0001 C CNN
+F 0 "#PWR029" H 10800 6200 50  0001 C CNN
 F 1 "+3.3V" H 10800 6490 50  0000 C CNN
 F 2 "" H 10800 6350 50  0001 C CNN
@@
 $EndComp
 $Comp
-L GND #PWR035
+L GND #PWR030
 U 1 1 58C60CEB
 P 11500 6800
-F 0 "#PWR035" H 11500 6550 50  0001 C CNN
+F 0 "#PWR030" H 11500 6550 50  0001 C CNN
 F 1 "GND" H 11500 6650 50  0000 C CNN
 F 2 "" H 11500 6800 50  0001 C CNN
@@
 SW[E]
 $Comp
-L GND #PWR036
+L GND #PWR031
 U 1 1 58C612CA
 P 13200 8650
-F 0 "#PWR036" H 13200 8400 50  0001 C CNN
+F 0 "#PWR031" H 13200 8400 50  0001 C CNN
 F 1 "GND" H 13200 8500 50  0000 C CNN
 F 2 "" H 13200 8650 50  0001 C CNN
@@
 +3.3V
 $Comp
-L GND #PWR037
+L GND #PWR032
 U 1 1 58CB109D
 P 9500 3200
-F 0 "#PWR037" H 9500 2950 50  0001 C CNN
+F 0 "#PWR032" H 9500 2950 50  0001 C CNN
 F 1 "GND" H 9500 3050 50  0000 C CNN
 F 2 "" H 9500 3200 50  0001 C CNN
@@
 $EndComp
 $Comp
-L GND #PWR038
+L GND #PWR033
 U 1 1 58CB10A3
 P 10000 3200
-F 0 "#PWR038" H 10000 2950 50  0001 C CNN
+F 0 "#PWR033" H 10000 2950 50  0001 C CNN
 F 1 "GND" H 10000 3050 50  0000 C CNN
 F 2 "" H 10000 3200 50  0001 C CNN
@@
 CTS_FTDI
 $Comp
-L +3.3V #PWR039
+L +3.3V #PWR034
 U 1 1 58C8A5C0
 P 15300 3700
-F 0 "#PWR039" H 15300 3550 50  0001 C CNN
+F 0 "#PWR034" H 15300 3550 50  0001 C CNN
 F 1 "+3.3V" V 15200 3750 50  0000 C CNN
 F 2 "" H 15300 3700 50  0001 C CNN
@@
 $EndComp
 $Comp
-L GND #PWR040
+L GND #PWR035
 U 1 1 58CB8882
 P 10050 9650
-F 0 "#PWR040" H 10050 9400 50  0001 C CNN
+F 0 "#PWR035" H 10050 9400 50  0001 C CNN
 F 1 "GND" H 10050 9500 50  0000 C CNN
 F 2 "" H 10050 9650 50  0001 C CNN
@@
 	10050 9600 10050 9650
 $Comp
-L GND #PWR041
+L GND #PWR036
 U 1 1 58CB8BE9
 P 10050 9300
-F 0 "#PWR041" H 10050 9050 50  0001 C CNN
+F 0 "#PWR036" H 10050 9050 50  0001 C CNN
 F 1 "GND" H 10050 9150 50  0000 C CNN
 F 2 "" H 10050 9300 50  0001 C CNN
@@
 $EndComp
 $Comp
-L GND #PWR042
+L GND #PWR037
 U 1 1 58CB8C8E
 P 10050 8950
-F 0 "#PWR042" H 10050 8700 50  0001 C CNN
+F 0 "#PWR037" H 10050 8700 50  0001 C CNN
 F 1 "GND" H 10050 8800 50  0000 C CNN
 F 2 "" H 10050 8950 50  0001 C CNN
@@
 $EndComp
 $Comp
-L GND #PWR043
+L GND #PWR038
 U 1 1 58CB8D80
 P 10050 8600
-F 0 "#PWR043" H 10050 8350 50  0001 C CNN
+F 0 "#PWR038" H 10050 8350 50  0001 C CNN
 F 1 "GND" H 10050 8450 50  0000 C CNN
 F 2 "" H 10050 8600 50  0001 C CNN
@@
 	1    0    0    -1
 $EndComp
+$Comp
+L +3.3V #PWR039
+U 1 1 58CEC3CC
+P 8500 5550
+F 0 "#PWR039" H 8500 5400 50  0001 C CNN
+F 1 "+3.3V" H 8500 5700 50  0000 C CNN
+F 2 "" H 8500 5550 50  0001 C CNN
+F 3 "" H 8500 5550 50  0001 C CNN
+	1    8500 5550
+	1    0    0    -1
+$EndComp
+$Comp
+L +3.3V #PWR040
+U 1 1 58CECF76
+P 7850 3450
+F 0 "#PWR040" H 7850 3300 50  0001 C CNN
+F 1 "+3.3V" H 7850 3600 50  0000 C CNN
+F 2 "" H 7850 3450 50  0001 C CNN
+F 3 "" H 7850 3450 50  0001 C CNN
+	1    7850 3450
+	1    0    0    -1
+$EndComp
+$Comp
+L +3.3V #PWR041
+U 1 1 58CED8E1
+P 8650 1850
+F 0 "#PWR041" H 8650 1700 50  0001 C CNN
+F 1 "+3.3V" H 8650 2000 50  0000 C CNN
+F 2 "" H 8650 1850 50  0001 C CNN
+F 3 "" H 8650 1850 50  0001 C CNN
+	1    8650 1850
+	1    0    0    -1
+$EndComp
+$Comp
+L +3.3V #PWR042
+U 1 1 58CED986
+P 9100 1600
+F 0 "#PWR042" H 9100 1450 50  0001 C CNN
+F 1 "+3.3V" H 9100 1750 50  0000 C CNN
+F 2 "" H 9100 1600 50  0001 C CNN
+F 3 "" H 9100 1600 50  0001 C CNN
+	1    9100 1600
+	1    0    0    -1
+$EndComp
+$Comp
+L +3.3V #PWR043
+U 1 1 58CEDA2B
+P 9550 1350
+F 0 "#PWR043" H 9550 1200 50  0001 C CNN
+F 1 "+3.3V" H 9550 1500 50  0000 C CNN
+F 2 "" H 9550 1350 50  0001 C CNN
+F 3 "" H 9550 1350 50  0001 C CNN
+	1    9550 1350
+	1    0    0    -1
+$EndComp
