File: kicad/kinetis.sch (KiCad schematic (older format))
At the start: 75 parts, among them J1 CONN_01X16, J2 CONN_01X16, J3 CONN_01X16, J4 CONN_01X16, J5 USB_Micro_B, J6 FTDI_Connector, J7 JLink_SWD_20pin, M1 #4-40 Mounting Hole, M2 #4-40 Mounting Hole, M3 #4-40 Mounting Hole, M4 #4-40 Mounting Hole, SW1 SPST, SW2 SPST, SW3 SPST, SW4 SPST, SW5 SPST, SW6 DPDT, U1 MKL16Z64VLH4, U2 LM1117-ADJ, Y1 12.000 MHz

Commit message: Renamed 5V input net
Connections:
- net labels added: PWR_IN
Changed lines of the file:
@@
 Wire Wire Line
 	9100 1650 9100 1700
+Text Label 13270 2000 2    60   ~ 0
+PWR_IN
 $EndSCHEMATC

Commit message: Back-annotated schematic from PCB.
This commit back-annotates the schematic from the PCB, and
includes the script that was used to do it.
Parts:
- renumbered C14 to C1, C4 to C10, C3 to C11, C17 to C12, C7 to C13, C1 to C14, C5 to C15, C15 to C17, C13 to C2, C9 to C3, C8 to C4, C10 to C5, C12 to C6, C11 to C7, C2 to C8, C6 to C9, D6 to D1, D5 to D2, D7 to D3, D9 to D4, D8 to D5, D1 to D6, D2 to D7, D3 to D8, D4 to D9, J5 to J1, J7 to J2, J1 to J3, J6 to J5, J2 to J6, J3 to J7, M3 to M1, M4 to M2, M2 to M3, M1 to M4, R24 to R1, R31 to R10, R30 to R11, R29 to R12, R1 to R13, R2 to R14, R3 to R15, R4 to R16, R10 to R17, R9 to R18, R8 to R19, R23 to R2, R17 to R20, R16 to R21, R7 to R22, R6 to R23, R5 to R24, R22 to R25, R21 to R26, R28 to R27, R25 to R28, R26 to R3, R27 to R4, R13 to R5, R14 to R6, R12 to R7, R11 to R8, R32 to R9, SW6 to SW1, SW1 to SW2, SW2 to SW3, SW3 to SW4, SW4 to SW5, SW5 to SW6, U2 to U1, U1 to U2

Commit message: Re-applied annotation
Parts:
- renumbered C5 to C1, C9 to C10, C14 to C12, C8 to C13, C15 to C14, C13 to C15, C6 to C2, C7 to C4, C4 to C5, C1 to C6, C10 to C7, C2 to C8, C12 to C9, D4 to D1, D5 to D2, D1 to D3, D2 to D4, D3 to D5, J5 to J1, J3 to J2, J1 to J3, J6 to J4, J2 to J5, J4 to J6, M3 to M2, M2 to M3, R20 to R1, R16 to R10, R13 to R11, R14 to R12, R5 to R13, R6 to R14, R25 to R15, R26 to R16, R3 to R17, R4 to R18, R7 to R19, R8 to R20, R17 to R21, R18 to R22, R19 to R23, R22 to R24, R23 to R25, R24 to R26, R10 to R3, R9 to R4, R11 to R5, R15 to R6, R21 to R7, R12 to R8, R1 to R9, SW3 to SW2, SW2 to SW3, SW5 to SW4, SW4 to SW5

Commit message: Changed USB connector. Fixed soldermask clearance settings.
This commit changes the USB connector from an SMT-only connector
to one with some through-hole mounting tabs. This should help to
provide mechanical ruggedness for the board.

This commit also fixed the soldermask clearance settings so that the
USB connector and Kinets both have soldermask in-between the pins.
Parts:
- J3: footprint custom_footprints:10118192-0001LF -> custom_footprints:10118193-0001LF; Manufacturer PN 10118192-0001LF -> 10118193-0001LF
Changed lines of the file:
@@
 LIBS:opto
 LIBS:atmel
-LIBS:kinetis-cache
 EELAYER 26 0
 EELAYER END
@@
 F 0 "J3" H 12500 5810 60  0000 C CNN
 F 1 "USB_Micro_B" H 12730 5730 60  0000 C CNN
-F 2 "custom_footprints:10118192-0001LF" H 12850 5600 60  0001 C CNN
+F 2 "custom_footprints:10118193-0001LF" H 12850 5600 60  0001 C CNN
 F 3 "" H 12850 5600 60  0001 C CNN
 F 4 "Amphenol FCI" H 12350 6200 60  0001 C CNN "Manufacturer"
-F 5 "10118192-0001LF" H 12350 6300 60  0001 C CNN "Manufacturer PN"
+F 5 "10118193-0001LF" H 12350 6300 60  0001 C CNN "Manufacturer PN"
 	1    12450 5650
 	1    0    0    -1

Commit message: Misc tweaks
Parts:
- added C13, C17, C8: 0.1uF, custom_footprints:SM_0603, symbol C
- renumbered C9 to C10, C10 to C11, C11 to C12, C13 to C14, C14 to C15, C15 to C16, C12 to C18, C16 to C19, C17 to C20, C8 to C9
Connections:
- wire segments 314 -> 326
Other:
- moved on the sheet: C18, R10, R6

Commit message: Cosmetic tweaks. Added copper thieving.
This commit adds ground-referenced copper thieving to the top layer
of the PCB, and also makes a whole bunch of cosmetic changes, including
a logo on the PCB and schematic, and infoblocks for the CCA and PCB.
Changed lines of the file:
@@
 encoding utf-8
 Sheet 1 1
-Title ""
-Date ""
-Rev ""
-Comp ""
+Title "The Ripper: Kinetis KL016 Eval Board"
+Date "2017-03-24"
+Rev "1.0"
+Comp "Hoboshop"
 Comment1 ""
 Comment2 ""
@@
 L HOLE M4
 U 1 1 58CB7CC4
-P 10300 8550
-F 0 "M4" H 10473 8596 50  0000 L CNN
-F 1 "#4-40 Mounting Hole" H 10473 8505 50  0000 L CNN
-F 2 "custom_footprints:4_40_Hole" H 10300 8550 50  0001 C CNN
-F 3 "" H 10300 8750 50  0001 C CNN
-F 4 "(none)" H 10300 9025 60  0001 C CNN "Manufacturer"
-F 5 "(none)" H 10300 8900 60  0001 C CNN "Manufacturer PN"
-	1    10300 8550
+P 9920 8560
+F 0 "M4" H 10093 8606 50  0000 L CNN
+F 1 "#4-40 Mounting Hole" H 10093 8515 50  0000 L CNN
+F 2 "custom_footprints:4_40_Hole" H 9920 8560 50  0001 C CNN
+F 3 "" H 9920 8760 50  0001 C CNN
+F 4 "(none)" H 9920 9035 60  0001 C CNN "Manufacturer"
+F 5 "(none)" H 9920 8910 60  0001 C CNN "Manufacturer PN"
+	1    9920 8560
 	1    0    0    -1
 $EndComp
@@
 L HOLE M2
 U 1 1 58CB7E94
-P 10300 8900
-F 0 "M2" H 10473 8946 50  0000 L CNN
-F 1 "#4-40 Mounting Hole" H 10473 8855 50  0000 L CNN
-F 2 "custom_footprints:4_40_Hole" H 10300 8900 50  0001 C CNN
-F 3 "" H 10300 9100 50  0001 C CNN
-F 4 "(none)" H 10300 9375 60  0001 C CNN "Manufacturer"
-F 5 "(none)" H 10300 9250 60  0001 C CNN "Manufacturer PN"
-	1    10300 8900
+P 9920 8910
+F 0 "M2" H 10093 8956 50  0000 L CNN
+F 1 "#4-40 Mounting Hole" H 10093 8865 50  0000 L CNN
+F 2 "custom_footprints:4_40_Hole" H 9920 8910 50  0001 C CNN
+F 3 "" H 9920 9110 50  0001 C CNN
+F 4 "(none)" H 9920 9385 60  0001 C CNN "Manufacturer"
+F 5 "(none)" H 9920 9260 60  0001 C CNN "Manufacturer PN"
+	1    9920 8910
 	1    0    0    -1
 $EndComp
@@
 L HOLE M1
 U 1 1 58CB7F7E
-P 10300 9250
-F 0 "M1" H 10473 9296 50  0000 L CNN
-F 1 "#4-40 Mounting Hole" H 10473 9205 50  0000 L CNN
-F 2 "custom_footprints:4_40_Hole" H 10300 9250 50  0001 C CNN
-F 3 "" H 10300 9450 50  0001 C CNN
-F 4 "(none)" H 10300 9725 60  0001 C CNN "Manufacturer"
-F 5 "(none)" H 10300 9600 60  0001 C CNN "Manufacturer PN"
-	1    10300 9250
+P 9920 9260
+F 0 "M1" H 10093 9306 50  0000 L CNN
+F 1 "#4-40 Mounting Hole" H 10093 9215 50  0000 L CNN
+F 2 "custom_footprints:4_40_Hole" H 9920 9260 50  0001 C CNN
+F 3 "" H 9920 9460 50  0001 C CNN
+F 4 "(none)" H 9920 9735 60  0001 C CNN "Manufacturer"
+F 5 "(none)" H 9920 9610 60  0001 C CNN "Manufacturer PN"
+	1    9920 9260
 	1    0    0    -1
 $EndComp
@@
 L HOLE M3
 U 1 1 58CB8044
-P 10300 9600
-F 0 "M3" H 10473 9646 50  0000 L CNN
-F 1 "#4-40 Mounting Hole" H 10473 9555 50  0000 L CNN
-F 2 "custom_footprints:4_40_Hole" H 10300 9600 50  0001 C CNN
-F 3 "" H 10300 9800 50  0001 C CNN
-F 4 "(none)" H 10300 10075 60  0001 C CNN "Manufacturer"
-F 5 "(none)" H 10300 9950 60  0001 C CNN "Manufacturer PN"
-	1    10300 9600
+P 9920 9610
+F 0 "M3" H 10093 9656 50  0000 L CNN
+F 1 "#4-40 Mounting Hole" H 10093 9565 50  0000 L CNN
+F 2 "custom_footprints:4_40_Hole" H 9920 9610 50  0001 C CNN
+F 3 "" H 9920 9810 50  0001 C CNN
+F 4 "(none)" H 9920 10085 60  0001 C CNN "Manufacturer"
+F 5 "(none)" H 9920 9960 60  0001 C CNN "Manufacturer PN"
+	1    9920 9610
 	1    0    0    -1
 $EndComp
@@
 L GND #PWR035
 U 1 1 58CB8882
-P 10050 9650
-F 0 "#PWR035" H 10050 9400 50  0001 C CNN
-F 1 "GND" H 10050 9500 50  0000 C CNN
-F 2 "" H 10050 9650 50  0001 C CNN
-F 3 "" H 10050 9650 50  0001 C CNN
-	1    10050 9650
+P 9670 9660
+F 0 "#PWR035" H 9670 9410 50  0001 C CNN
+F 1 "GND" H 9670 9510 50  0000 C CNN
+F 2 "" H 9670 9660 50  0001 C CNN
+F 3 "" H 9670 9660 50  0001 C CNN
+	1    9670 9660
 	-1   0    0    -1
 $EndComp
@@
 L GND #PWR036
 U 1 1 58CB8BE9
-P 10050 9300
-F 0 "#PWR036" H 10050 9050 50  0001 C CNN
-F 1 "GND" H 10050 9150 50  0000 C CNN
-F 2 "" H 10050 9300 50  0001 C CNN
-F 3 "" H 10050 9300 50  0001 C CNN
-	1    10050 9300
+P 9670 9310
+F 0 "#PWR036" H 9670 9060 50  0001 C CNN
+F 1 "GND" H 9670 9160 50  0000 C CNN
+F 2 "" H 9670 9310 50  0001 C CNN
+F 3 "" H 9670 9310 50  0001 C CNN
+	1    9670 9310
 	-1   0    0    -1
 $EndComp
@@
 L GND #PWR037
 U 1 1 58CB8C8E
-P 10050 8950
-F 0 "#PWR037" H 10050 8700 50  0001 C CNN
-F 1 "GND" H 10050 8800 50  0000 C CNN
-F 2 "" H 10050 8950 50  0001 C CNN
-F 3 "" H 10050 8950 50  0001 C CNN
-	1    10050 8950
+P 9670 8960
+F 0 "#PWR037" H 9670 8710 50  0001 C CNN
+F 1 "GND" H 9670 8810 50  0000 C CNN
+F 2 "" H 9670 8960 50  0001 C CNN
+F 3 "" H 9670 8960 50  0001 C CNN
+	1    9670 8960
 	-1   0    0    -1
 $EndComp
@@
 L GND #PWR038
 U 1 1 58CB8D80
-P 10050 8600
-F 0 "#PWR038" H 10050 8350 50  0001 C CNN
-F 1 "GND" H 10050 8450 50  0000 C CNN
-F 2 "" H 10050 8600 50  0001 C CNN
-F 3 "" H 10050 8600 50  0001 C CNN
-	1    10050 8600
+P 9670 8610
+F 0 "#PWR038" H 9670 8360 50  0001 C CNN
+F 1 "GND" H 9670 8460 50  0000 C CNN
+F 2 "" H 9670 8610 50  0001 C CNN
+F 3 "" H 9670 8610 50  0001 C CNN
+	1    9670 8610
 	-1   0    0    -1
 $EndComp
@@
 	1600 8900 1900 8900
 Wire Wire Line
-	10100 9600 10050 9600
-Wire Wire Line
-	10050 9600 10050 9650
-Wire Wire Line
-	10100 8550 10050 8550
-Wire Wire Line
-	10050 8550 10050 8600
-Wire Wire Line
-	10100 8900 10050 8900
-Wire Wire Line
-	10050 8900 10050 8950
-Wire Wire Line
-	10100 9250 10050 9250
-Wire Wire Line
-	10050 9250 10050 9300
-Wire Notes Line
-	9900 8300 11400 8300
-Wire Notes Line
-	9900 9900 11400 9900
-Wire Notes Line
-	9900 8300 9900 9900
-Wire Notes Line
-	11400 9900 11400 8300
+	9720 9610 9670 9610
+Wire Wire Line
+	9670 9610 9670 9660
+Wire Wire Line
+	9720 8560 9670 8560
+Wire Wire Line
+	9670 8560 9670 8610
+Wire Wire Line
+	9720 8910 9670 8910
+Wire Wire Line
+	9670 8910 9670 8960
+Wire Wire Line
+	9720 9260 9670 9260
+Wire Wire Line
+	9670 9260 9670 9310
+Wire Notes Line
+	9520 8310 11020 8310
+Wire Notes Line
+	9520 9910 11020 9910
+Wire Notes Line
+	9520 8310 9520 9910
+Wire Notes Line
+	11020 9910 11020 8310
 Wire Wire Line
 	13950 1950 14025 1950
@@
 	7700 3500 7910 3500
 $Comp
-L GND #PWR?
+L GND #PWR049
 U 1 1 58D449EE
 P 1940 1980
-F 0 "#PWR?" H 1940 1730 50  0001 C CNN
+F 0 "#PWR049" H 1940 1730 50  0001 C CNN
 F 1 "GND" H 1940 1830 50  0000 C CNN
 F 2 "" H 1940 1980 50  0001 C CNN
@@
 $EndComp
 $Comp
-L +3.3V #PWR?
+L +3.3V #PWR050
 U 1 1 58D449FC
 P 1940 1560
-F 0 "#PWR?" H 1940 1410 50  0001 C CNN
+F 0 "#PWR050" H 1940 1410 50  0001 C CNN
 F 1 "+3.3V" H 1940 1710 50  0000 C CNN
 F 2 "" H 1940 1560 50  0001 C CNN

Commit message: Footprint and copper tweaks.
This commit changes out the USB connector footprint for a tweaked
version with thru-holes instead of slots. It also fixes a minor
silkscreen bug in the SM_0805 package, and lengthens the CCA
title block.

Additionally, the GND pours on top/bottom were pulled back from the
PCB edge by 0.020".
Parts:
- J3: footprint custom_footprints:10118193-0001LF -> custom_footprints:10118193-0001LF_noslots
Changed lines of the file:
@@
 F 0 "J3" H 12500 5810 60  0000 C CNN
 F 1 "USB_Micro_B" H 12730 5730 60  0000 C CNN
-F 2 "custom_footprints:10118193-0001LF" H 12850 5600 60  0001 C CNN
+F 2 "custom_footprints:10118193-0001LF_noslots" H 12850 5600 60  0001 C CNN
 F 3 "" H 12850 5600 60  0001 C CNN
 F 4 "Amphenol FCI" H 12350 6200 60  0001 C CNN "Manufacturer"

Commit message: Fixed the manufacturer/part-numers for resistors.
This commit changes the MFR and MFR PN for four 200-ohm resistors
which were accidentally called out with 0.1-ohm part numbers. Oops.
Parts:
- R13, R14, R25, R26: Manufacturer CTS -> Yageo; Manufacturer PN 73L3R10J -> RC0805FR-07200RL
Changed lines of the file:
@@
 LIBS:opto
 LIBS:atmel
-LIBS:kinetis-cache
 EELAYER 26 0
 EELAYER END
@@
 F 2 "custom_footprints:SM_0805" V 1380 5600 50  0001 C CNN
 F 3 "" H 1450 5800 50  0001 C CNN
-F 4 "CTS" H 1450 5900 60  0001 C CNN "Manufacturer"
-F 5 "73L3R10J" H 1450 6000 60  0001 C CNN "Manufacturer PN"
+F 4 "Yageo" H 1450 5900 60  0001 C CNN "Manufacturer"
+F 5 "RC0805FR-07200RL" H 1450 6000 60  0001 C CNN "Manufacturer PN"
 	1    1450 5600
 	1    0    0    -1
@@
 F 2 "custom_footprints:SM_0805" V 1380 5900 50  0001 C CNN
 F 3 "" H 1450 6100 50  0001 C CNN
-F 4 "CTS" H 1450 6200 60  0001 C CNN "Manufacturer"
-F 5 "73L3R10J" H 1450 6300 60  0001 C CNN "Manufacturer PN"
+F 4 "Yageo" H 1450 6200 60  0001 C CNN "Manufacturer"
+F 5 "RC0805FR-07200RL" H 1450 6300 60  0001 C CNN "Manufacturer PN"
 	1    1450 5900
 	1    0    0    -1
@@
 F 2 "custom_footprints:SM_0805" V 1380 9200 50  0001 C CNN
 F 3 "" H 1450 9400 50  0001 C CNN
-F 4 "CTS" H 1450 9500 60  0001 C CNN "Manufacturer"
-F 5 "73L3R10J" H 1450 9600 60  0001 C CNN "Manufacturer PN"
+F 4 "Yageo" H 1450 9500 60  0001 C CNN "Manufacturer"
+F 5 "RC0805FR-07200RL" H 1450 9600 60  0001 C CNN "Manufacturer PN"
 	1    1450 9200
 	1    0    0    -1
@@
 F 2 "custom_footprints:SM_0805" V 1380 8900 50  0001 C CNN
 F 3 "" H 1450 9100 50  0001 C CNN
-F 4 "CTS" H 1450 9200 60  0001 C CNN "Manufacturer"
-F 5 "73L3R10J" H 1450 9300 60  0001 C CNN "Manufacturer PN"
+F 4 "Yageo" H 1450 9200 60  0001 C CNN "Manufacturer"
+F 5 "RC0805FR-07200RL" H 1450 9300 60  0001 C CNN "Manufacturer PN"
 	1    1450 8900
 	1    0    0    -1
